Commit message: Update: Integrate gripper including UEDF

File: gen3_lite.urdf (robot description, URDF)
Before this commit: robot KR7108-URDF, 8 links, 7 joints
Links:
- added link GRIPPER_FRAME, mass 0.1395; collision mesh filename=meshes/GRIPPER_FRAME.STL; visual mesh filename=meshes/GRIPPER_FRAME.STL
- added link LEFT_FINGER_DIST, mass 0.010748; collision mesh filename=meshes/LEFT_FINGER_DIST.STL; visual mesh filename=meshes/LEFT_FINGER_DIST.STL
- added link LEFT_FINGER_PROX, mass 0.018385; collision mesh filename=meshes/LEFT_FINGER_PROX.STL; visual mesh filename=meshes/LEFT_FINGER_PROX.STL
- added link RIGHT_FINGER_DIST, mass 0.010748; collision mesh filename=meshes/RIGHT_FINGER_DIST.STL; visual mesh filename=meshes/RIGHT_FINGER_DIST.STL
- added link RIGHT_FINGER_PROX, mass 0.018385; collision mesh filename=meshes/RIGHT_FINGER_PROX.STL; visual mesh filename=meshes/RIGHT_FINGER_PROX.STL
Joints:
- removed joint END_EFFECTOR
- added joint END_EFFECTOR_FIXED: type fixed, parent END_EFFECTOR, child DUMMY, origin xyz=0 0 0.13 rpy=0 0 0
- added joint LEFT_BOTTOM: type revolute, parent GRIPPER_FRAME, child LEFT_FINGER_PROX, origin xyz=0 0.0305 0.070003 rpy=0 1.5708 0, axis 0 0 1, limit lower=-0.96 upper=0.09 effort=1000 velocity=1000
- added joint LEFT_TIP: type revolute, parent LEFT_FINGER_PROX, child LEFT_FINGER_DIST, origin xyz=-0.045636 -0.020423 6.9901E-05 rpy=0 0 0, axis 0 0 -1, limit lower=-0.21 upper=1.03 effort=1000 velocity=1000
- added joint RIGHT_BOTTOM: type revolute, parent GRIPPER_FRAME, child RIGHT_FINGER_PROX, origin xyz=0 -0.030501 0.070003 rpy=0 1.5708 0, axis 0 0 1, limit lower=-0.09 upper=0.96 effort=1000 velocity=1000
- added joint RIGHT_TIP: type revolute, parent RIGHT_FINGER_PROX, child RIGHT_FINGER_DIST, origin xyz=-0.045636 0.020423 0 rpy=0 0 0, axis 0 0 1, limit lower=-1.03 upper=0.21 effort=1000 velocity=1000
- added joint arm_to_gripper: type fixed, parent END_EFFECTOR, child GRIPPER_FRAME, origin xyz=0 0 0 rpy=0 0 0
